File: Hardware/FurbyBoard/hojas/motor.kicad_sch (KiCad schematic)
At the start: 31 parts, among them U5 TPS61089RNRR, U6 DRV8231ADSGR

Commit message: Fix: A2, R24 a 33 kΩ 0402 básica (C25779) en vez de 30 kΩ extended, con la E2 repetida
Revisión independiente de M3: el 30 kΩ 0402 (C25776) es extended en JLCPCB (3,07 USD de carga por
pedido) y el 33 kΩ 0402 (C25779, UNI-ROYAL 0402WGF3302TCE) es básica (API de JLCPCB, 2026-10-27:
2 540 677 en stock, 0,0019 USD). Lazo del TPS61089 con las ecuaciones 11-19 de SLVSD38C (VREF
1,212 V, GEA 190 µS, Rsense 0,08 Ω, L 1 µH ± 20 %, Cout 42-70 µF efectivos, VIN 2,7-4,4 V,
0,2-1 A): con 33 k fC 20-40 kHz, siempre < fSW/10 (96 kHz) y < fRHPZ/5 (26 kHz en la peor esquina),
margen de fase mínimo 78,8° (30 k: 79,9°) y de ganancia ≥ 16 dB. Misma posición, giro y huella;
C14 y C15 sin cambios.

- design.py: RES0402 con C25779 (base); R24 "33k". Esquema y PCB regenerados: el único cambio
  en la placa son las propiedades de R24 (Value, LCSC, JLC_Class, Description); el resto es
  idéntico salvo 44 vértices de relleno con diferencias de 1e-6 mm (misma área y trozos).
- sim/models/furby.lib: R24 33 k; drv8231a_motor.cir y arranque_brownout.cir repetidos: rizado
  de V6 con el motor bloqueado 119 mV pp (antes 130) y 18 mV pp en PWM (antes 19); el resto igual.
- Fabricación (make_fab.sh con el pcb-toolkit del venv): rellenos al día, ERC 0, DRC con paridad
  0/0/0, Gerber idénticos por geometría a los de e558d6a (solo cambian fechas y numeración de
  aperturas), taladros idénticos, BOM 52 líneas / 126 piezas con 18 extended (antes 19), CPL sin
  cambios, cpl-rotaciones PASS con 3 giro-sin-tabla (C25105 ×2, C25779).
- NOTAS (decisión A2 y cálculo del lazo), README de fabricación (coste 55,26 de carga, fila de
  R24, tabla de la BOM) y sim/RESULTADOS.md al día.

Co-Authored-By: Claude Fable 5.1 <noreply@anthropic.com>
Parts:
- R24: value 30k -> 33k; JLC_Class ext -> base; LCSC C25776 -> C25779
Changed lines of the file:
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@@
 			)
 		)
-		(property "Value" "30k"
+		(property "Value" "33k"
 			(at 90.4 124.19 0)
 			(show_name no)
@@
 			)
 		)
-		(property "Description" "Compensación (fc ≈ 20–30 kHz)"
+		(property "Description" "Compensación (fc ≈ 20–33 kHz)"
 			(at 88.9 127 0)
 			(hide yes)
@@
 			)
 		)
-		(property "LCSC" "C25776"
+		(property "LCSC" "C25779"
 			(at 88.9 127 0)
 			(hide yes)
@@
 			)
 		)
-		(property "JLC_Class" "ext"
+		(property "JLC_Class" "base"
 			(at 88.9 127 0)
 			(hide yes)
